Commit message: fix the arm (now points to the front of the robot

File: urdf/2wheels_with_arm.urdf (robot description, URDF)
Before this commit: robot 2wheels, 13 links, 12 joints
Joints:
- joint arm_to_laser: origin xyz=0 0 0.05 rpy=0 0 0 -> xyz=0 0 0.05 rpy=0 0 -1.5707

Commit message: Some changes to the arm, not good yet

File: urdf/2wheels_with_arm.urdf (robot description, URDF)
Before this commit: robot 2wheels, 13 links, 12 joints
Links:
- link arm_link_01: geometry collision cylinder length=0.06 radius=0.017; visual cylinder length=0.06 radius=0.017
- link arm_link_02: geometry collision cylinder length=0.06 radius=0.010; visual cylinder length=0.06 radius=0.010
- link arm_link_03: geometry collision cylinder length=0.06 radius=0.010; visual cylinder length=0.06 radius=0.010
Joints:
- joint arm_joint_01: origin xyz=0 0 0.05 rpy=0 0 0 -> xyz=0 0 0.04 rpy=0 0 0
- joint arm_joint_02: origin xyz=0 0 0.02 rpy=0 0 0 -> xyz=0 0 0.01 rpy=0 0 0
- joint arm_joint_03: axis 1 0 0 -> 1  0  0; origin xyz=0 0 0.02 rpy=0 0 0 -> xyz=0 0 0.04 rpy=0 0 0
- joint arm_to_laser: origin xyz=0 0 0.05 rpy=0 0 -1.5707 -> xyz=0 0 0.04 rpy=0 0 -1.5707

Commit message: Adapting 2wheels to work with nav2d

File: urdf/2wheels_with_arm.urdf (robot description, URDF)
Before this commit: robot 2wheels, 13 links, 12 joints
Links:
- removed link sensor_laser
- added link base_laser_link, mass 0.25; collision cylinder length=0.05 radius=0.05; visual cylinder length=0.05 radius=0.05
Joints:
- removed joint joint_sensor_laser
- added joint joint_base_laser_link: type fixed, parent base_link, child base_laser_link, origin xyz=0.0 0 0.07 rpy=0 0 0
- joint arm_to_laser: parent sensor_laser -> base_laser_link

Commit message: Rearranging everything it is almost o.k, I just need to fix the left part fo the gripper

File: urdf/2wheels_with_arm.urdf (robot description, URDF)
Before this commit: robot 2wheels, 13 links, 12 joints
Links:
- link arm_base_link: geometry collision box size=0.05 0.05 0.03; visual box size=0.05 0.05 0.03
- link arm_link_02: geometry collision box size=0.1 0.03 0.02; visual box size=0.1 0.03 0.02
- link arm_link_03: geometry collision box size=0.1 0.03 0.02; visual box size=0.1 0.03 0.02
- link arm_link_04: geometry collision box size=0.08 0.04 0.02; visual box size=0.08 0.04 0.02
- link right_grip_link: mass 0.005 -> 0.05
Joints:
- removed joint arm_to_laser
- added joint laser_to_arm_base: type fixed, parent base_laser_link, child arm_base_link, origin xyz=0 0 0.025 rpy=0 0 0
- joint arm_joint_01: origin xyz=0 0 0.04 rpy=0 0 0 -> xyz=0 0 0.03 rpy=0 0 0
- joint arm_joint_02: axis 1 0 0 -> 0 0 1; origin xyz=0 0 0.01 rpy=0 0 0 -> xyz=0 0 0.05 rpy=1.5707 0 0
- joint arm_joint_03: axis 1  0  0 -> 0  0  1; origin xyz=0 0 0.04 rpy=0 0 0 -> xyz=0.1 0 0 rpy=0 0 0
- joint arm_joint_04: axis 1 0 0 -> 0 0 1; origin xyz=0 0 0.02 rpy=0 0 0 -> xyz=0.1 0 0.0 rpy=0 1.570796 0
- joint left_grip_joint: axis -1 0 0 -> 0 0 1; origin xyz=-0.015 0.0 0.0 rpy=0 0 0 -> xyz=0.0 0.0 0 rpy=0 1.570796 0
- joint right_grip_joint: axis 1 0 0 -> 0 0 1; limit lower=-0.01 upper=0.035 effort=1000 velocity=6.5 -> lower=-0.04 upper=0.04 effort=1000 velocity=1.0; origin xyz=-0.015 0.0 0 rpy=0 0 0 -> xyz=-0.02 0 0 rpy=0 -1.570796 0

Commit message: The arm visual is ready, I still need to adjust the mass of the arm to make it remain still

File: urdf/2wheels_with_arm.urdf (robot description, URDF)
Before this commit: robot 2wheels, 13 links, 12 joints
Joints:
- joint left_grip_joint: limit lower=-0.01 upper=0.035 effort=1000 velocity=6.5 -> lower=0 upper=0.05 effort=1000 velocity=0.5; origin xyz=0.0 0.0 0 rpy=0 1.570796 0 -> xyz=0.0 0.0 0 rpy=3.14159 -1.570796 0
- joint right_grip_joint: limit lower=-0.04 upper=0.04 effort=1000 velocity=1.0 -> lower=0 upper=0.05 effort=1000 velocity=1.0; origin xyz=-0.02 0 0 rpy=0 -1.570796 0 -> xyz=0.0 0 0 rpy=0 -1.570796 0

Commit message: IS WORKINGgit status I added colors, modified masses and inertias, now it looks great.

File: urdf/2wheels_with_arm.urdf (robot description, URDF)
Before this commit: robot 2wheels, 13 links, 12 joints
Links:
- removed link camera_link
- added link camera1_link, mass 0.04; collision box size=0.03 0.05 0.03; visual box size=0.03 0.05 0.03
- link arm_link_04: geometry collision box size=0.08 0.04 0.02; visual box size=0.1 0.022 0.006
- link left_grip_link: mass 0.01 -> 0.001; geometry collision mesh filename=package://two_wheels_description/meshes/chain_link_grip_l.s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 scale=0.001 0.001 0.001; visual mesh filename=package://two_wheels_description/meshes/chain_link_grip_l.s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 scale=0.0005 0.0005 0.0005
- link right_grip_link: mass 0.05 -> 0.001; geometry collision mesh filename=package://two_wheels_description/meshes/chain_link_grip_r.s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 scale=0.001 0.001 0.001; visual mesh filename=package://two_wheels_description/meshes/chain_link_grip_r.s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 scale=0.0005 0.0005 0.0005
Joints:
- removed joint camera_joint
- added joint camera1_joint: type revolute, parent base_link, child camera1_link, origin xyz=0.11 0.0 0.04 rpy=0 0 0, axis 0 1 0, limit lower=-0.8 upper=0.3 effort=100000.0 velocity=0.2
- joint arm_joint_02: limit lower=-1.8 upper=1.8 effort=1000.0 velocity=0.2 -> lower=-0.1 upper=1.5707 effort=10000.0 velocity=0.2
- joint arm_joint_03: limit lower=-1.8 upper=1.8 effort=1000.0 velocity=0.2 -> lower=-0.1 upper=1.5707 effort=10000.0 velocity=0.2
- joint arm_joint_04: limit lower=-1.8 upper=1.8 effort=1000.0 velocity=0.5 -> lower=-1.8 upper=1.8 effort=10000.0 velocity=0.5
- joint left_grip_joint: limit lower=0 upper=0.05 effort=1000 velocity=0.5 -> lower=0 upper=0.05 effort=100000 velocity=0.4
- joint right_grip_joint: limit lower=0 upper=0.05 effort=1000 velocity=1.0 -> lower=0 upper=0.05 effort=100000 velocity=0.4

Commit message: Added some inclination (pitch) to the joint that connects the laser_link to the base_link to avoid having refections against the floor

File: urdf/2wheels_with_arm.urdf (robot description, URDF)
Before this commit: robot 2wheels, 13 links, 12 joints
Links:
- link caster_wheel: geometry collision sphere radius=0.0051; visual sphere radius=0.005
Joints:
- joint joint_base_laser_link: origin xyz=0.0 0 0.07 rpy=0 0 0 -> xyz=0.0 0 0.085 rpy=0 0.04 0

Commit message: smaller mass for the robot

File: urdf/2wheels_with_arm.urdf (robot description, URDF)
Before this commit: robot 2wheels, 13 links, 12 joints
Links:
- link base_link: mass 10.0 -> 6.0

Commit message: fixing misalignment of the laser that caused some errors when using the lidar data for mapping

File: urdf/2wheels_with_arm.urdf (robot description, URDF)
Before this commit: robot 2wheels, 13 links, 12 joints
Joints:
- joint joint_base_laser_link: origin xyz=0.0 0 0.085 rpy=0 0.04 0 -> xyz=0.0 0 0.085 rpy=0 0.0 0
- joint joint_caster: origin xyz=0.085 -0.008 -0.015 rpy=0 0 0 -> xyz=0.085 -0.008 -0.009 rpy=0 0 0

Commit message: fixing misalignment of the laser that caused some errors when using the lidar data for mapping

File: urdf/2wheels_with_arm.urdf (robot description, URDF)
Before this commit: robot 2wheels, 13 links, 12 joints
Joints:
- joint joint_base_laser_link: origin xyz=0.0 0 0.085 rpy=0 0.04 0 -> xyz=0.0 0 0.085 rpy=0 0.0 0

Commit message: changes to work in melodic

File: urdf/2wheels_with_arm.urdf (robot description, URDF)
Before this commit: robot 2wheels, 13 links, 12 joints
Links:
- link arm_link_01: mass 0.0125 -> 0.0025
- link arm_link_02: mass 0.0125 -> 0.0025
- link arm_link_03: mass 0.0125 -> 0.0025
- link arm_link_04: mass 0.0125 -> 0.0025
- link base_laser_link: mass 0.25 -> 0.05
- link left_grip_link: mass 0.001 -> 0.0001
- link right_grip_link: mass 0.001 -> 0.0001

Commit message: Solving the problem: the robot was turning in the opposite direction in ROS melodic

File: urdf/2wheels_with_arm.urdf (robot description, URDF)
Before this commit: robot 2wheels, 13 links, 12 joints
Joints:
- joint joint_caster: limit effort=1000 velocity=10 -> effort=10 velocity=10
