Commit message: Larger arm links and added damping factors to avoid the arm oscillations

File: urdf/arm.urdf (robot description, URDF)
Before this commit: robot robot, 9 links, 8 joints
Links:
- removed link arm_link_04
- added link gripper_base, mass 0.0025; collision box size=0.8 0.4 0.2; visual box size=0.2 0.22 0.06
- link arm_link_01: mass 0.0025 -> 0.25; geometry collision cylinder length=0.6 radius=0.17; visual cylinder length=0.6 radius=0.17
- link arm_link_02: mass 0.0025 -> 0.25; geometry collision box size=0.1 0.3 0.2; visual box size=1.0 0.3 0.2
- link arm_link_03: mass 0.0025 -> 0.025; geometry collision box size=1.0 0.3 0.2; visual box size=1 0.3 0.2
- link base_link: geometry collision box size=0.5 0.5 0.3; visual box size=0.5 0.5 0.3
- link left_grip_link: geometry collision mesh filename=package://two_wheels_description/meshes/chain_link_grip_l.s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 scale=0.001 0.001 0.001; visual mesh filename=package://two_wheels_description/meshes/chain_link_grip_l.s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 scale=0.005 0.005 0.005
- link right_grip_link: geometry collision mesh filename=package://two_wheels_description/meshes/chain_link_grip_r.s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 scale=0.001 0.001 0.001; visual mesh filename=package://two_wheels_description/meshes/chain_link_grip_r.s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 scale=0.005 0.005 0.005
Joints:
- joint arm_joint_01: limit lower=-3.14 upper=3.14 effort=1000.0 velocity=0.2 -> lower=-3.1416 upper=3.1416 effort=1000.0 velocity=1.0; origin xyz=0 0 0.03 rpy=0 0 0 -> xyz=0 0 0.3 rpy=0 0 0
- joint arm_joint_02: limit lower=-0.1 upper=1.5707 effort=10000.0 velocity=0.2 -> lower=-0.1 upper=1.57079632 effort=10000.0 velocity=1.0; origin xyz=0 0 0.05 rpy=1.5707 0 0 -> xyz=0 0 0.5 rpy=1.57079632 0 0
- joint arm_joint_03: limit lower=-0.1 upper=1.5707 effort=10000.0 velocity=0.2 -> lower=-1.57079632 upper=1.57079632 effort=10000.0 velocity=1.0; origin xyz=0.1 0 0 rpy=0 0 0 -> xyz=1 0 0 rpy=0 0 0
- joint arm_joint_04: child arm_link_04 -> gripper_base; limit lower=-1.8 upper=1.8 effort=10000.0 velocity=0.5 -> lower=-1.8 upper=1.8 effort=100.0 velocity=0.5; origin xyz=0.1 0 0.0 rpy=0 1.570796 0 -> xyz=1.0 0 0.0 rpy=0 1.570796 0
- joint left_grip_joint: parent arm_link_04 -> gripper_base
- joint right_grip_joint: limit lower=0 upper=0.05 effort=100000 velocity=0.4 -> lower=0 upper=0.1 effort=100000 velocity=0.4; parent arm_link_04 -> gripper_base

Commit message: The camera of the arm is now pointing down from the top of the workspace

File: urdf/arm.urdf (robot description, URDF)
Before this commit: robot robot, 9 links, 8 joints
Links:
- link arm_link_02: geometry collision box size=0.6 0.15 0.1; visual box size=0.6 0.15 0.1
- link arm_link_03: geometry collision box size=0.6 0.15 0.1; visual box size=0.6 0.15 0.1
- link base_link: geometry collision box size=0.5 0.5 0.1; visual box size=0.5 0.5 0.1
- link camera1_link: mass 0.04 -> 0.00000001; geometry collision box size=0.1 0.15 0.1; visual box size=0.1 0.15 0.1
Joints:
- joint arm_joint_01: origin xyz=0 0 0.3 rpy=0 0 0 -> xyz=0 0 0.1 rpy=0 0 0
- joint arm_joint_03: limit lower=-1.57079632 upper=1.57079632 effort=10000.0 velocity=1.0 -> lower=-1.57079632 upper=1.57079632 effort=100000.0 velocity=1.0; origin xyz=1 0 0 rpy=0 0 0 -> xyz=0.6 0 0 rpy=0 0 0
- joint arm_joint_04: origin xyz=1.0 0 0.0 rpy=0 1.570796 0 -> xyz=0.6 0 0.0 rpy=0 1.570796 0
- joint camera1_joint: limit lower=-0.8 upper=0.3 effort=100000.0 velocity=0.2 -> (none); origin xyz=0.11 0.0 0.04 rpy=0 0 0 -> xyz=1.1 0.0 1.9 rpy=0 1.5707 0; type revolute -> fixed

Commit message: Fixing the gripper size

File: urdf/arm.urdf (robot description, URDF)
Before this commit: robot robot, 9 links, 8 joints
Links:
- link gripper_base: geometry collision box size=0.2 0.05 0.01; visual box size=0.2 0.05 0.01
- link left_grip_link: geometry collision mesh filename=package://two_wheels_description/meshes/chain_link_grip_l.s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 scale=0.001 0.001 0.001; visual mesh filename=package://two_wheels_description/meshes/chain_link_grip_l.s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 scale=0.001 0.001 0.001
- link right_grip_link: geometry collision mesh filename=package://two_wheels_description/meshes/chain_link_grip_r.s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 scale=0.001 0.001 0.001; visual mesh filename=package://two_wheels_description/meshes/chain_link_grip_r.s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 scale=0.001 0.001 0.001
Joints:
- joint arm_joint_01: limit lower=-3.1416 upper=3.1416 effort=1000.0 velocity=1.0 -> lower=-3.1416 upper=3.1416 effort=1000.0 velocity=2.0
- joint arm_joint_02: limit lower=-0.1 upper=1.57079632 effort=10000.0 velocity=1.0 -> lower=-0.1 upper=1.57079632 effort=10000.0 velocity=2.0
- joint arm_joint_03: limit lower=-1.57079632 upper=1.57079632 effort=100000.0 velocity=1.0 -> lower=-1.57079632 upper=1.57079632 effort=100000.0 velocity=2.0
- joint arm_joint_04: limit lower=-1.8 upper=1.8 effort=100.0 velocity=0.5 -> lower=-3.1416 upper=3.1416 effort=100000.0 velocity=2.0
- joint right_grip_joint: limit lower=0 upper=0.1 effort=100000 velocity=0.4 -> lower=0 upper=0.05 effort=100000 velocity=0.4

Commit message: Adding a world with a table to put the arm.urdf

File: urdf/arm.urdf (robot description, URDF)
Before this commit: robot robot, 9 links, 8 joints
Joints:
- joint camera1_joint: origin xyz=1.1 0.0 1.9 rpy=0 1.5707 0 -> xyz=1.0 0.0 1.9 rpy=0 1.5707 0

Commit message: changed the pid parameters of the arm simulation to make joint 2 to achieve the required angle correctly

File: urdf/arm.urdf (robot description, URDF)
Before this commit: robot robot, 9 links, 8 joints
Links:
- link arm_link_01: mass 0.25 -> 0.025
- link base_link: mass 0.05 -> 5.0
Joints:
- joint arm_joint_02: limit lower=-0.1 upper=1.57079632 effort=10000.0 velocity=2.0 -> lower=-0.7 upper=1.57079632 effort=10000.0 velocity=2.0
