Commit message: Solving the state_publisher' executable is deprecated warning and The root link base_link has an inertia specified in the URDF, but KDL does not support a root link with an inertia warning

File: urdf/2wheels_simple.urdf (robot description, URDF)
Before this commit: robot 2wheels, 6 links, 5 joints
Links:
- added link dummy_base
Joints:
- added joint dummy joint: type fixed, parent dummy_base, child base_link, origin xyz=0 0 0 rpy=0 0 0

File: urdf/2wheels_with_arm.urdf (robot description, URDF)
Before this commit: robot 2wheels, 13 links, 12 joints
Links:
- added link dummy_base
Joints:
- added joint dummy joint: type fixed, parent dummy_base, child base_link, origin xyz=0 0 0 rpy=0 0 0

Commit message: change the 2wheels simulation, now the dummy_base link is the base_link and the link for the chassis is called like that (chassis_link)

File: urdf/2wheels_simple.urdf (robot description, URDF)
Before this commit: robot 2wheels, 7 links, 6 joints
Links:
- removed link dummy_base
- added link chassis_link, mass 6.0; collision box size=0.18 0.2 0.06; visual mesh filename=package://two_wheels_description/meshes/robotmodel.dae
- link base_link: mass 6.0 -> None; geometry 
Joints:
- joint camera1_joint: parent base_link -> chassis_link
- joint dummy joint: child base_link -> chassis_link; parent dummy_base -> base_link
- joint joint_base_laser_link: parent base_link -> chassis_link
- joint joint_caster: parent base_link -> chassis_link
- joint joint_left_wheel: parent base_link -> chassis_link
- joint joint_right_wheel: parent base_link -> chassis_link

File: urdf/2wheels_with_arm.urdf (robot description, URDF)
Before this commit: robot 2wheels, 14 links, 13 joints
Links:
- removed link dummy_base
- added link chassis_link, mass 6.0; collision box size=0.18 0.2 0.05; visual mesh filename=package://two_wheels_description/meshes/robotmodel.dae
- link base_link: mass 6.0 -> None; geometry 
Joints:
- joint camera1_joint: parent base_link -> chassis_link
- joint dummy joint: child base_link -> chassis_link; parent dummy_base -> base_link
- joint joint_base_laser_link: parent base_link -> chassis_link
- joint joint_caster: parent base_link -> chassis_link
- joint joint_left_wheel: parent base_link -> chassis_link
- joint joint_right_wheel: parent base_link -> chassis_link

Commit message: Changed two_wheels model to make it move more smoothly, deleted the mesh to make it less computationally expensive

File: urdf/2wheels_simple.urdf (robot description, URDF)
Before this commit: robot 2wheels, 7 links, 6 joints
Links:
- link caster_wheel: geometry collision sphere radius=0.01; visual sphere radius=0.01
- link chassis_link: geometry collision box size=0.18 0.2 0.06; visual box size=0.18 0.2 0.06
- link link_left_wheel: geometry collision cylinder length=0.01 radius=0.035; visual cylinder length=0.01 radius=0.035
- link link_right_wheel: geometry collision cylinder length=0.01 radius=0.035; visual cylinder length=0.01 radius=0.035
Joints:
- joint joint_caster: limit effort=1000 velocity=10 -> (none); origin xyz=0.085 -0.008 -0.015 rpy=0 0 0 -> xyz=0.085 -0.008 -0.02 rpy=0 0 0

Commit message: moving the robot's caster wheel to the back and the actuated wheels to the front

File: urdf/2wheels_simple.urdf (robot description, URDF)
Before this commit: robot 2wheels, 7 links, 6 joints
Joints:
- joint joint_caster: origin xyz=0.085 -0.008 -0.02 rpy=0 0 0 -> xyz=-0.075 0.0 -0.02 rpy=0 0 0
- joint joint_left_wheel: origin xyz=-0.0572 0.11  0.006 rpy=1.57079632 0  0 -> xyz=0.0572 0.11  0.006 rpy=1.57079632 0  0
- joint joint_right_wheel: origin xyz=-0.0572 -0.11 0.006 rpy=-1.57079632 0  0 -> xyz=0.0572 -0.11 0.006 rpy=-1.57079632 0  0

Commit message: Modifying the mass of the chassis to make it lighter

File: urdf/2wheels_simple.urdf (robot description, URDF)
Before this commit: robot 2wheels, 7 links, 6 joints
Links:
- link base_laser_link: mass 0.25 -> 0.2
- link chassis_link: mass 6.0 -> 0.4
